File: buoy-c/buoy-c.sch (KiCad schematic (older format))
At the start: 91 parts, among them J1 UJ31-CH-G2-SMT-TR, J10 Conn_01x06_Male, J11 TERM-BLK-2P, J14 Conn_01x09_Male, J2 BAT-HLD-001-THM, J3 Conn_01x02_Male, J4 U.FL-R-SMT-1_10_, J5 BH-18650-PC, J7 Conn_01x02_Male, J8 Conn_01x03_Male, J9 U.FL-R-SMT-1_10_, Q1 MMBT2222LT1G, Q2 MMBT2222LT1G, Q3 MMBT2222LT1G, U1 ATGM332D-5N31, U10 LTC2954ITS8-1#TRPBF, U2 LTC3113EFE#TRPBF, U3 TP4056, U4 ESP32-WROOM-32D, U5 FT260S-U, U6 TPS61030PWPR, U7 RFM95W-915S2, U8 DS3231M+TRL

Commit message: Added gerber files
Parts:
- C15, C16, C18, C22: Manufacturer Samsung Electro-Mechanics -> YAGEO; Manufacturer Part Number (none) -> CC0805KKX7R7BB105; Supplier Part Number 1 1276-1275-1-ND -> 311-1365-1-ND
- R27: Supplier Part Number RR12P180KDCT-ND -> (none); Supplier Part Number 1 (none) -> RR12P180KDCT-ND
- U8: Supplier Part Number DS3231M+TRLCT-ND -> (none); Supplier Part Number 1 (none) -> DS3231M+TRLCT-ND
Changed lines of the file:
@@
 Sheet 1 1
 Title "Buoy C - Leonardo Ward"
-Date "2021-08-22"
+Date "2021-09-02"
 Rev "1.0"
 Comp ""
@@
 $EndComp
 $Comp
-L C-1uF-0805:1uF C16
-U 1 1 612F63BB
-P 10500 1600
-F 0 "C16" H 10615 1646 50  0000 L CNN
-F 1 "1uF" H 10615 1555 50  0000 L CNN
-F 2 "Capacitor_SMD:C_0805_2012Metric" H 12300 1800 100 0001 C CNN
-F 3 "http://www.samsungsem.com/kr/support/product-search/mlcc/CL21B105KPFNNNE.jsp" H 10500 1600 100 0001 C CNN
-F 4 "Samsung Electro-Mechanics" H 12100 1600 100 0001 C CNN "Manufacturer"
-F 5 "CL21B105KPFNNNE" H 14000 1600 100 0001 C CNN "Manufacturer_Part_Number"
-F 6 "Digi-Key" H 11350 1450 100 0001 C CNN "Supplier 1"
-F 7 "1276-1275-1-ND" H 12550 1450 100 0001 C CNN "Supplier Part Number 1"
-	1    10500 1600
-	1    0    0    -1
-$EndComp
-$Comp
-L C-1uF-0805:1uF C18
-U 1 1 612F7340
-P 11000 2700
-F 0 "C18" H 11115 2746 50  0000 L CNN
-F 1 "1uF" H 11115 2655 50  0000 L CNN
-F 2 "Capacitor_SMD:C_0805_2012Metric" H 12800 2900 100 0001 C CNN
-F 3 "http://www.samsungsem.com/kr/support/product-search/mlcc/CL21B105KPFNNNE.jsp" H 11000 2700 100 0001 C CNN
-F 4 "Samsung Electro-Mechanics" H 12600 2700 100 0001 C CNN "Manufacturer"
-F 5 "CL21B105KPFNNNE" H 14500 2700 100 0001 C CNN "Manufacturer_Part_Number"
-F 6 "Digi-Key" H 11850 2550 100 0001 C CNN "Supplier 1"
-F 7 "1276-1275-1-ND" H 13050 2550 100 0001 C CNN "Supplier Part Number 1"
-	1    11000 2700
-	1    0    0    -1
-$EndComp
-$Comp
 L R-10K-0805:10K R23
 U 1 1 612F7EB3
@@
 F 5 "DS3231M+TRL" H 12250 6100 50  0001 C CNN "Manufacturer Part Number"
 F 6 "Digi-Key" H 11400 6000 50  0001 C CNN "Supplier 1"
-F 7 "DS3231M+TRLCT-ND" H 12100 6000 50  0001 C CNN "Supplier Part Number"
+F 7 "DS3231M+TRLCT-ND" H 10450 5800 50  0001 C CNN "Supplier Part Number 1"
 	1    10450 5800
 	1    0    0    -1
 $EndComp
-$Comp
-L C-1uF-0805:1uF C15
-U 1 1 61302292
-P 9100 5500
-F 0 "C15" H 9215 5546 50  0000 L CNN
-F 1 "1uF" H 9215 5455 50  0000 L CNN
-F 2 "Capacitor_SMD:C_0805_2012Metric" H 10900 5700 100 0001 C CNN
-F 3 "http://www.samsungsem.com/kr/support/product-search/mlcc/CL21B105KPFNNNE.jsp" H 9100 5500 100 0001 C CNN
-F 4 "Samsung Electro-Mechanics" H 10700 5500 100 0001 C CNN "Manufacturer"
-F 5 "CL21B105KPFNNNE" H 12600 5500 100 0001 C CNN "Manufacturer_Part_Number"
-F 6 "Digi-Key" H 9950 5350 100 0001 C CNN "Supplier 1"
-F 7 "1276-1275-1-ND" H 11150 5350 100 0001 C CNN "Supplier Part Number 1"
-	1    9100 5500
-	1    0    0    -1
-$EndComp
 Text GLabel 1800 5500 0    50   Output ~ 0
 BAT-CR2032
@@
 F 5 "RR1220P-184-D" H 11150 7700 50  0001 C CNN "Manufacturer Part Number"
 F 6 "Digi-Key" H 10600 7600 50  0001 C CNN "Supplier 1"
-F 7 "RR12P180KDCT-ND" H 11200 7600 50  0001 C CNN "Supplier Part Number"
+F 7 "RR12P180KDCT-ND" H 10100 7600 50  0001 C CNN "Supplier Part Number 1"
 	1    10100 7600
 	1    0    0    -1
@@
 F 2 "Capacitor_SMD:C_0805_2012Metric" H 15500 2400 100 0001 C CNN
 F 3 "http://www.samsungsem.com/kr/support/product-search/mlcc/CL21B105KPFNNNE.jsp" H 13700 2200 100 0001 C CNN
-F 4 "Samsung Electro-Mechanics" H 15300 2200 100 0001 C CNN "Manufacturer"
+F 4 "YAGEO" H 15300 2200 100 0001 C CNN "Manufacturer"
 F 5 "CL21B105KPFNNNE" H 17200 2200 100 0001 C CNN "Manufacturer_Part_Number"
 F 6 "Digi-Key" H 14550 2050 100 0001 C CNN "Supplier 1"
-F 7 "1276-1275-1-ND" H 15750 2050 100 0001 C CNN "Supplier Part Number 1"
+F 7 "311-1365-1-ND" H 15750 2050 100 0001 C CNN "Supplier Part Number 1"
+F 8 "CC0805KKX7R7BB105" H 13700 2200 50  0001 C CNN "Manufacturer Part Number"
 	1    13700 2200
 	1    0    0    -1
@@
 Wire Wire Line
 	7400 9450 7050 9450
+$Comp
+L C-1uF-0805:1uF C18
+U 1 1 612F7340
+P 11000 2700
+F 0 "C18" H 11115 2746 50  0000 L CNN
+F 1 "1uF" H 11115 2655 50  0000 L CNN
+F 2 "Capacitor_SMD:C_0805_2012Metric" H 12800 2900 100 0001 C CNN
+F 3 "http://www.samsungsem.com/kr/support/product-search/mlcc/CL21B105KPFNNNE.jsp" H 11000 2700 100 0001 C CNN
+F 4 "YAGEO" H 12600 2700 100 0001 C CNN "Manufacturer"
+F 5 "CL21B105KPFNNNE" H 14500 2700 100 0001 C CNN "Manufacturer_Part_Number"
+F 6 "Digi-Key" H 11850 2550 100 0001 C CNN "Supplier 1"
+F 7 "311-1365-1-ND" H 13050 2550 100 0001 C CNN "Supplier Part Number 1"
+F 8 "CC0805KKX7R7BB105" H 11000 2700 50  0001 C CNN "Manufacturer Part Number"
+	1    11000 2700
+	1    0    0    -1
+$EndComp
+$Comp
+L C-1uF-0805:1uF C15
+U 1 1 61302292
+P 9100 5500
+F 0 "C15" H 9215 5546 50  0000 L CNN
+F 1 "1uF" H 9215 5455 50  0000 L CNN
+F 2 "Capacitor_SMD:C_0805_2012Metric" H 10900 5700 100 0001 C CNN
+F 3 "http://www.samsungsem.com/kr/support/product-search/mlcc/CL21B105KPFNNNE.jsp" H 9100 5500 100 0001 C CNN
+F 4 "YAGEO" H 10700 5500 100 0001 C CNN "Manufacturer"
+F 5 "CL21B105KPFNNNE" H 12600 5500 100 0001 C CNN "Manufacturer_Part_Number"
+F 6 "Digi-Key" H 9950 5350 100 0001 C CNN "Supplier 1"
+F 7 "311-1365-1-ND" H 11150 5350 100 0001 C CNN "Supplier Part Number 1"
+F 8 "CC0805KKX7R7BB105" H 9100 5500 50  0001 C CNN "Manufacturer Part Number"
+	1    9100 5500
+	1    0    0    -1
+$EndComp
+$Comp
+L C-1uF-0805:1uF C16
+U 1 1 612F63BB
+P 10500 1600
+F 0 "C16" H 10615 1646 50  0000 L CNN
+F 1 "1uF" H 10615 1555 50  0000 L CNN
+F 2 "Capacitor_SMD:C_0805_2012Metric" H 12300 1800 100 0001 C CNN
+F 3 "http://www.samsungsem.com/kr/support/product-search/mlcc/CL21B105KPFNNNE.jsp" H 10500 1600 100 0001 C CNN
+F 4 "YAGEO" H 12100 1600 100 0001 C CNN "Manufacturer"
+F 5 "CL21B105KPFNNNE" H 14000 1600 100 0001 C CNN "Manufacturer_Part_Number"
+F 6 "Digi-Key" H 11350 1450 100 0001 C CNN "Supplier 1"
+F 7 "311-1365-1-ND" H 12550 1450 100 0001 C CNN "Supplier Part Number 1"
+F 8 "CC0805KKX7R7BB105" H 10500 1600 50  0001 C CNN "Manufacturer Part Number"
+	1    10500 1600
+	1    0    0    -1
+$EndComp
 $EndSCHEMATC
